File: ice40/milliLearn-ice40/milliLearn-ice40.brd (EAGLE design)
At the start: 160 x 100 mm, 177 parts, among them J1 SFV24R-2STE1HLF, J2 10118194-0001LF, J3 SM04B-SRSS-TB(LF)(SN), U1 AP7366-W5-7, U10 AP7366-W5-7, U11 DSC6111CI2A-012.0000, U12 SPH0645LM4H-B, U13 SPH0645LM4H-B, U2 DSC6111CI2A-012.0000, U3 AP7366-W5-7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

Commit message: pcb-ng board wip
Parts:
- removed SW3: (no value), milliLearn-ice40:TE_FSMJSMA
- moved C14 210.4 mm to (25.4, 39.5), turned to 180 degrees
- moved JP27 207.4 mm to (43.7, 86.5)
- moved JP29 207.4 mm to (64.1, 86.5)
- moved JP33 207.4 mm to (69.1, 92.9)
- moved JP34 207.4 mm to (73.2, 92.9)
- moved JP28 204.9 mm to (98.8, 86.5)
- moved JP30 204.9 mm to (78.4, 86.8)
- moved JP35 204.9 mm to (103.8, 92.8)
- moved JP36 204.9 mm to (107.9, 92.8)
- moved C15 199.9 mm to (26.8, 46.5), turned to 90 degrees
- moved R29 155.0 mm to (80.8, 61.9), turned to 270 degrees
- moved R28 154.4 mm to (79.8, 61.9), turned to 270 degrees
- moved C16 147.0 mm to (-21.3, 80.4)
- moved C44 142.2 mm to (65.5, 58.8), flipped to the bottom, turned to 180 degrees
- moved C43 139.2 mm to (65.2, 57.8), flipped to the bottom
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Connections:
- removed net I2S_DATA: JP40.27, U12.P$6, U13.P$6, U8.20
- removed net ICE40_+1V2: C34.2, C35.2, C36.2, C37.2, JP5.2, R25.1, U8.30, U8.5
- removed net MEM2_CIPO: JP27.3, JP28.3, JP41.7, U8.47
- removed net MEM2_COPI: JP29.7, JP30.7, JP41.11, U8.2
- removed net N$34: LED6.A, R38.2
- new net ICE40_+1V2_CORE: C34.2, C35.2, C36.2, C37.2, JP20.2, U8.30, U8.5
- new net ICE40_+1V2_PLL: JP5.2, R25.1
- new net MEM2_CIPO1: JP27.3, JP41.7, U8.47
- new net MEM2_CIPO2: JP28.3, U8.4
- new net MEM2_COPI1: JP29.7, JP41.11, U8.2
- new net MEM2_COPI2: JP30.7, U8.44
- net +1V2: now also JP20.1
- net +1V2_METERED: now also JP20.3
- net +1V8: no longer JP20.1
- net +1V8_METERED: no longer JP20.3
- net GND: now also LED6.C; no longer SW3.P$3, SW3.P$4
- net HM01B0_INT: now also LED3.C; no longer SW3.P$1, SW3.P$2
- net ICE40_FLASH_CIPO: now also JP40.27, U12.P$6, U13.P$6; no longer LED3.C
- net ICE40_GPIO4: no longer LED6.C, U8.4
- net ICE40_GPIO43: now also LED6.A, R38.2
- net ICE40_OSC_12M: now also U8.20; no longer U8.44
- net ICE40_OSC_VCC: no longer JP20.2
Routing:
- net HM01B0_D1: track 1.62 -> 13.5 mm
- net N$3: track 0.00 -> 6.50 mm
- net ICE40_+1V2: track 5.22 -> 0.00 mm, vias 1 -> 0
- net ICE40_+1V2_PLL: track 0.00 -> 3.64 mm, vias 0 -> 1
- net ICE40_VCCIO2: track 0.00 -> 3.03 mm, vias 0 -> 1
- net HM01B0_SCL: track 17.0 -> 19.6 mm, vias 0 -> 2
- net HM01B0_SDA: track 17.7 -> 19.8 mm
- net +3V3_METERED: track 0.00 -> 1.74 mm
- net ICE40_+1V2_CORE: track 0.00 -> 0.81 mm
Other:
- board size 160 x 100 mm -> 160 x 110 mm
- board text added: "+1v2"
- board text added: "+1v8"
- board text added: "+2v8"
- board text added: "+3v3"
- board text added: "100mV / mA"
- board text added: "gnd"
