File: ice40/milliLearn-ice40-pcbng/milliLearn-ice40-pcbng.brd (EAGLE design)
At the start: 70 x 39 mm, 162 parts, among them J1 SFV24R-2STE1HLF, J2 10118194-0001LF, J3 SM04B-SRSS-TB(LF)(SN), U1 AP7366-W5-7, U10 AP7366-W5-7, U11 DSC6111CI2A-012.0000, U12 SPH0645LM4H-B, U13 SPH0645LM4H-B, U14 CY15B104Q-LHXI, U15 CY15B104Q-LHXI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

Commit message: routing for pcbng variant wip
Parts:
- removed C27, C28, C30, C48: 22u, rcl:C1210
- removed LED6: (no value), led:CHIPLED_0603
- removed R36: 1k, milliLearn-ice40:R0402_COMPACT
- added JP31: (no value), pinhead:1X02
- added TP0, TP1, TP10, TP11, TP12, TP13, TP14, TP15, TP16, TP17, TP18, TP2, TP3, TP4, TP5, TP6, TP7, TP8, TP9: TPTP10SQ, testpad:TP10SQ
- moved JP28 237.8 mm to (25.6, 30.6), flipped to the bottom, turned to 0 degrees
- moved JP30 230.9 mm to (59.0, 12.4), flipped to the bottom, turned to 0 degrees
- moved JP27 226.8 mm to (25.6, 32.2), flipped to the bottom, turned to 0 degrees
- moved JP29 211.9 mm to (63.0, 26.4), flipped to the bottom, turned to 0 degrees
- moved JP26 199.6 mm to (45.8, 30.3), flipped to the bottom
- moved JP23 195.0 mm to (27.1, 8.70), flipped to the bottom, turned to 90 degrees
- moved JP24 190.6 mm to (42.8, 9.40), flipped to the bottom, turned to 90 degrees
- moved JP25 188.7 mm to (45.8, 32.0), flipped to the bottom
- moved JP4 154.4 mm to (25.1, 16.8), flipped to the bottom, turned to 270 degrees
- moved JP22 153.8 mm to (67.0, 4.75), flipped to the bottom
- moved JP17 153.7 mm to (47.1, 18.2), flipped to the bottom, turned to 0 degrees
- moved JP16 145.5 mm to (47.1, 16.1), flipped to the bottom, turned to 0 degrees
- moved JP21 129.6 mm to (50.1, 12.3), turned to 90 degrees
- moved JP19 125.7 mm to (47.5, 9.05), flipped to the bottom, turned to 90 degrees
- moved JP20 121.6 mm to (30.6, 24.4), flipped to the bottom, turned to 0 degrees
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Connections:
- removed net I2S_WS: JP40.29, U12.P$1, U13.P$1, U8.21
- removed net ICE40_GPIO4: JP41.15
- removed net N$32: LED4.A, R36.2
- new net I2S_DATA: JP40.25, U12.P$6, U13.P$6, U8.18
- new net N$34: U13.P$1
- new net N$35: U13.P$4
- new net N$36: U12.P$4
- new net N$37: U12.P$1
- net +1V2_METERED: now also C26.1, R24.2, U9.2; no longer C24.1, C27.1, R22.2, U9.9
- net +1V8_METERED: no longer C28.1
- net +2V8_METERED: no longer C48.1
- net +3V3: now also U13.P$2; no longer R36.1
- net +3V3_METERED: now also C24.1, R22.2, U9.9; no longer C26.1, C30.1, R24.2, U9.2
- net GND: now also JP31.2, LED5.C, TP0.TP, TP17.TP, TP18.TP; no longer C27.2, C28.2, C30.2, C48.2, LED6.C
- net HM01B0_D0: now also TP9.TP
- net HM01B0_D1: now also TP1.TP
- net HM01B0_D2: now also TP6.TP
- net HM01B0_D3: now also TP2.TP
- net HM01B0_D4: now also TP7.TP
- net HM01B0_D5: now also TP14.TP
- net HM01B0_D6: now also TP13.TP
- net HM01B0_D7: now also TP8.TP
- net HM01B0_HS: now also TP10.TP
- net HM01B0_INT: now also TP12.TP
- net HM01B0_MCK: now also TP5.TP
- net HM01B0_PCLK: now also TP11.TP
- net HM01B0_SCL: now also TP15.TP
- net HM01B0_SDA: now also TP16.TP
- net HM01B0_TRIG: now also LED4.C, TP4.TP; no longer LED5.C
- net HM01B0_VS: now also TP3.TP
- net ICE40_CRESETB: now also JP31.1
- net ICE40_FLASH_CIPO: now also JP40.9; no longer JP40.21, JP40.27, U12.P$6, U13.P$6
- net ICE40_FLASH_COPI: now also JP40.5; no longer JP40.15, LED4.C
- net ICE40_FLASH_PS: now also JP40.1; no longer JP40.19
- net ICE40_FLASH_SCK: now also JP40.3; no longer JP40.17, U12.P$4, U13.P$4
- net ICE40_GPIO43: now also LED5.A; no longer LED6.A
- net ICE40_OSC_12M: now also JP40.23; no longer JP41.1
- net MEM1_!HOLD: now also JP40.17, U8.10; no longer JP40.13, U8.13
- net MEM1_!WP: now also JP40.15, U8.7; no longer JP40.11, U8.12
- net MEM1_CIPO: now also JP40.7, U8.6; no longer JP40.9, U8.11
- net MEM1_COPI: now also JP40.21, U8.12; no longer JP40.25, U8.19
- net MEM1_PS1: now also JP40.11; no longer JP40.5
- net MEM1_PS2: now also JP40.13, U8.13; no longer JP40.7, U8.10
- net MEM1_SCK: now also JP40.19, U8.11; no longer JP40.23, U8.18
- net MEM2_!WP: now also U8.2; no longer JP41.9, U8.48
- net MEM2_CIPO1: now also U8.45; no longer JP41.7, U8.47
- net MEM2_CIPO2: now also U8.48; no longer U8.4
- net MEM2_COPI1: now also U8.46; no longer JP41.11, U8.2
- net MEM2_COPI2: now also U8.4; no longer U8.44
- net MEM2_PS1: now also U8.44; no longer JP41.3, U8.45
- net MEM2_PS2: now also U8.47; no longer JP41.5, U8.46
- net MEM2_SCK: no longer JP41.13
- net MIC2_VCC: no longer U13.P$2
- net N$33: now also LED4.A; no longer LED5.A
- net QWIIC_SCL: now also JP40.27, U8.21; no longer JP40.3, U8.7
- net QWIIC_SDA: now also JP40.29, U8.19; no longer JP40.1, U8.6
Routing:
- net +3V3: track 5.32 -> 216.7 mm, vias 0 -> 13
- net +3V3_METERED: track 14.3 -> 191.3 mm, vias 1 -> 12
- net +2V8: track 5.34 -> 106.6 mm, vias 0 -> 1
- net +2V8_METERED: track 11.0 -> 111.5 mm, vias 1 -> 3
- net ICE40_GPIO43: track 0.00 -> 68.3 mm, vias 0 -> 2
- net +1V8_METERED: track 5.07 -> 71.7 mm, vias 1 -> 7
- net +1V8: track 5.39 -> 64.0 mm, vias 0 -> 5
- net ICE40_CRESETB: track 0.00 -> 57.9 mm, vias 0 -> 3
- net ICE40_FLASH_SCK: track 2.48 -> 56.4 mm, vias 0 -> 6
- net MEM1_CIPO: track 0.00 -> 44.4 mm, vias 0 -> 2
- net ICE40_FLASH_CIPO: track 14.5 -> 57.3 mm, vias 0 -> 3
- net +1V2_METERED: track 4.29 -> 46.4 mm, vias 1 -> 4
- net QWIIC_SCL: track 0.00 -> 41.4 mm, vias 0 -> 3
- net QWIIC_SDA: track 0.00 -> 41.2 mm, vias 0 -> 2
- net MEM1_!WP: track 0.00 -> 38.5 mm, vias 0 -> 2
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
Commit message: first pass of routing done
Parts:
- C1: value (none) -> 1u
- moved JP12 7.57 mm to (13.8, 35.4)
- moved JP15 7.57 mm to (10.3, 35.4)
- moved JP10 7.57 mm to (20.8, 35.4)
- moved JP11 7.57 mm to (17.3, 35.4)
- moved JP22 6.10 mm to (67.0, 10.8)
- moved TP17 3.92 mm to (56.8, 24.4)
- moved C49 1.77 mm to (49.0, 6.80), turned to 90 degrees
- moved TP18 1.68 mm to (56.8, 17.2)
Connections:
- net N$23 renamed MEAS_1V2
- net N$24 renamed MEAS_1V8
- net N$25 renamed MEAS_3V3
- net N$26 renamed MEAS_2V8
- removed net N$34: U13.P$1
- removed net N$35: U13.P$4
- removed net N$36: U12.P$4
- removed net N$37: U12.P$1
- net ICE40_FLASH_CIPO: now also U12.P$1, U13.P$1
- net ICE40_FLASH_SCK: now also U12.P$4, U13.P$4
- net MEM2_!WP: now also JP41.5
- net MEM2_CIPO1: now also JP41.3
- net MEM2_CIPO2: now also JP41.11
- net MEM2_COPI1: now also JP41.7
- net MEM2_COPI2: now also JP41.15
- net MEM2_PS1: now also JP41.1
- net MEM2_PS2: now also JP41.9
- net MEM2_SCK: now also JP41.13
Routing:
- net HM01B0_TRIG: track 16.5 -> 72.9 mm, vias 1 -> 3
- net HM01B0_INT: track 18.9 -> 64.2 mm, vias 1 -> 3
- net I2S_DATA: track 21.2 -> 56.9 mm, vias 1 -> 2
- net ICE40_FLASH_CIPO: track 57.3 -> 92.6 mm, vias 3 -> 6
- net ICE40_FLASH_SCK: track 56.4 -> 88.4 mm, vias 6 -> 7
- net MEM2_PS1: track 10.9 -> 24.2 mm
- net MEM2_CIPO1: track 12.5 -> 23.4 mm, vias 0 -> 1
- net MEM2_!WP: track 22.6 -> 31.2 mm
- net MEM2_CIPO2: track 6.93 -> 15.5 mm
- net MEAS_1V2: track 1.93 -> 9.80 mm
- net MEM2_SCK: track 25.8 -> 33.1 mm
- net MEM2_COPI1: track 12.0 -> 18.9 mm
- net MEM2_COPI2: track 17.2 -> 23.7 mm, vias 1 -> 0
- net QWIIC_+3V3: track 10.0 -> 16.1 mm
- net MEAS_1V8: track 8.38 -> 13.5 mm
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Other:
- board text added: "10"
- board text added: "11"
- board text added: "12"
- board text added: "13"
- board text added: "14"
- board text added: "15"
- board text added: "16"
- board text added: "17"
- board text added: "18"
- board text added: "19"
- board text added: "1V2"
- board text added: "1V8"
- board text added: "2"
- board text added: "20"
- board text added: "21"
- board text added: "2V8"
- board text added: "3"
- board text added: "3V3"
- board text added: "4"
- board text added: "44"
- board text added: "45"
- board text added: "46"
- board text added: "47"
- board text added: "48"
- board text added: "6"
- board text added: "7"
- board text added: "9"
- board text added: "CAM_ANA"
- board text added: "CAM_IO"
- board text added: "CFG_MEM"
- board text added: "D0"
- board text added: "D1"
- board text added: "D2"
- board text added: "D3"
- board text added: "D4"
- board text added: "D5"
- board text added: "D6"
- board text added: "D7"
- board text added: "GND"
- board text added: "HSYNC"
- board text added: "ICE40_CORE"
- board text added: "ICE_2V5"
- board text added: "ICE_PLL"
- board text added: "IGNR"
- board text added: "INT"
- board text added: "Ka Moamoa"
- board text added: "MCK"
- board text added: "MEAS"
- board text added: "MEM1_1"
- board text added: "MEM1_2"
- board text added: "MEM2_1"
- board text added: "MEM2_2"
- board text added: "MIC1"
- board text added: "MIC2"
- board text added: "OSC"
- board text added: "PCLK"
- board text added: "QWIIC"
- board text added: "SCL"
- board text added: "SDA"
- board text added: "SJ5376"
- board text added: "Solder jumpers on the bottom determine which components are included in current measurement at top-left of board. IGNR = don't measure; MEAS = do measure"
- board text added: "Sparkfun QWIIC"
- board text added: "TRIG"
- board text added: "VCCIO0"
- board text added: "VCCIO1"
- board text added: "VCCIO2"
- board text added: "VSYNC"
- board text added: "foot"
- board text added: "milliLearn/iCE40"
