File: ice40/milliLearn-ice40-pcbng/milliLearn-ice40-pcbng.sch (EAGLE design)
At the start: 176 parts, among them J1 SFV24R-2STE1HLF, J2 10118194-0001LF, J3 SM04B-SRSS-TB(LF)(SN), U1 AP7366-W5-7, U10 AP7366-W5-7, U11 DSC6111CI2A-012.0000, U12 SPH0645LM4H-B, U13 SPH0645LM4H-B, U2 DSC6111CI2A-012.0000, U3 AP7366-W5-7, U4 AP7366-W5-7, U5 MICROBUILDER_FT232HQ, U6 MICROCHIP_93LC76B, U7 MT25QL128ABA1EW7, U8 ICE40UP5K/3K-SG48, U9 INA4180A4IPWR

Commit message: pcb-ng board wip
Parts:
- removed JP31, JP32, JP33, JP34, JP35, JP36, JP37, JP38: (no value), pinhead:PINHD-1X3
- removed JP39: (no value), pinhead:PINHD-2X17
- removed SJ1, SJ10, SJ11, SJ12, SJ13, SJ14, SJ15, SJ16, SJ17, SJ2, SJ3, SJ4, SJ5, SJ6, SJ7, SJ8, SJ9: JUMPER-SMT_2_NC_PASTE_NO-SILK, SparkFun-Jumpers:JUMPER-SMT_2_NC_PASTE_NO-SILK
- added C55, C56, C59, C61: 100n, milliLearn-ice40:C0402_COMPACT
- added C57, C58, C60, C62: 1u, milliLearn-ice40:C0402_COMPACT
- added U14, U15: CY15B104Q-LHXI, milliLearn-ice40:CY15B104Q-LHXI
- added U16, U17: AT25QF641B-SHB-T, milliLearn-ice40:AT25QF641B-SHB-T
- JP13, JP14, JP16, JP17, JP19, JP22, JP4, JP5, JP6, JP7, JP8: value (none) -> JUMPER-SMT_3_1-NC_PASTE_NO-SILK; device pinhead:PINHD-1X3 -> milliLearn-ice40:JUMPER-SMT_3_1-NC_PASTE_NO-SILK
- JP20, JP9: value (none) -> JUMPER-SMT_3_NO_NO-SILK; device pinhead:PINHD-1X3 -> milliLearn-ice40:JUMPER-SMT_3_NO_NO-SILK
- JP21: value (none) -> JUMPER-SMT_2_NO_NO-SILK; device pinhead:PINHD-1X2 -> milliLearn-ice40:JUMPER-SMT_2_NO_NO-SILK
- JP23, JP24, JP25, JP27, JP29, JP30: value (none) -> JUMPER-SMT_3_1-NC_PASTE_NO-SILK; device pinhead:PINHD-1X8 -> milliLearn-ice40:JUMPER-SMT_3_1-NC_PASTE_NO-SILK
- JP26, JP28: value (none) -> JUMPER-SMT_3_NO_NO-SILK; device pinhead:PINHD-1X8 -> milliLearn-ice40:JUMPER-SMT_3_NO_NO-SILK
Connections:
- removed net N$35: JP39.1, SJ1.2
- removed net N$36: JP39.3, SJ2.2
- removed net N$37: JP39.5, SJ3.2
- removed net N$38: JP39.7, SJ4.2
- removed net N$39: JP39.9, SJ5.2
- removed net N$40: JP39.11, SJ6.2
- removed net N$41: JP39.13, SJ7.2
- removed net N$42: JP39.15, SJ8.2
- removed net N$43: JP39.17, SJ9.2
- removed net N$44: JP39.19, SJ10.2
- removed net N$45: JP39.21, SJ11.2
- removed net N$46: JP39.23, SJ12.2
- removed net N$47: JP39.25, SJ13.2
- removed net N$48: JP39.27, SJ14.2
- removed net N$49: JP39.29, SJ15.2
- removed net N$50: JP39.31, SJ16.2
- removed net N$51: JP39.33, SJ17.2
- net +1V2: now also JP6.1; no longer JP20.1
- net +1V2_METERED: now also C24.1, C27.1, JP6.3, R22.2; no longer C26.1, C30.1, JP20.3, R24.2
- net +1V8: now also JP13.1, JP16.3, JP20.3, JP26.3, JP28.3; no longer JP14.1, JP16.1, JP34.1, JP36.1, JP9.1
- net +1V8_METERED: now also JP13.3, JP16.1, JP20.1, JP26.1, JP28.1; no longer JP14.3, JP16.3, JP34.3, JP36.3, JP9.3
- net +2V8: now also JP17.3; no longer JP17.1
- net +2V8_METERED: now also JP17.1; no longer JP17.3
- net +3V3: now also JP14.1, JP19.3, JP22.3, JP23.3, JP24.3, JP25.3, JP27.3, JP29.1, JP30.3, JP7.3, JP9.3; no longer JP13.1, JP19.1, JP22.1, JP31.1, JP32.1, JP33.1, JP35.1, JP37.1, JP38.1, JP6.1, JP7.1
- net +3V3_METERED: now also C26.1, C30.1, JP14.3, JP19.1, JP22.1, JP23.1, JP24.1, JP25.1, JP27.1, JP29.3, JP30.1, JP7.1, JP9.1, R24.2; no longer C24.1, C27.1, JP13.3, JP19.3, JP22.3, JP31.3, JP32.3, JP33.3, JP35.3, JP37.3, JP38.3, JP6.3, JP7.3, R22.2
- net GND: now also C55.P$1, C56.P$1, C57.P$1, C58.P$1, C59.P$1, C60.P$1, C61.P$1, C62.P$1, U14.VSS, U15.VSS, U16.GND, U16.PAD, U17.GND, U17.PAD; no longer JP23.2, JP23.4, JP23.6, JP23.7, JP23.8, JP24.2, JP24.4, JP24.6, JP24.7, JP24.8, JP25.2, JP25.4, JP25.6, JP25.8, JP26.2, JP26.4, JP26.6, JP26.8, JP27.2, JP27.4, JP27.6, JP27.7, JP27.8, JP28.2, JP28.4, JP28.6, JP28.7, JP28.8, JP29.2, JP29.4, JP29.6, JP29.8, JP30.2, JP30.4, JP30.6, JP30.8, JP39.10, JP39.12, JP39.14, JP39.16, JP39.18, JP39.2, JP39.20, JP39.22, JP39.24, JP39.26, JP39.28, JP39.30, JP39.32, JP39.34, JP39.4, JP39.6, JP39.8
- net HM01B0_D0: no longer SJ9.1
- net HM01B0_D1: no longer SJ1.1
- net HM01B0_D2: no longer SJ6.1
- net HM01B0_D3: no longer SJ2.1
- net HM01B0_D4: no longer SJ7.1
- net HM01B0_D5: no longer SJ14.1
- net HM01B0_D6: no longer SJ13.1
- net HM01B0_D7: no longer SJ8.1
- net HM01B0_HS: no longer SJ10.1
- net HM01B0_INT: no longer SJ12.1
- net HM01B0_MCK: no longer SJ5.1
- net HM01B0_PCLK: no longer SJ11.1
- net HM01B0_SCL: no longer SJ15.1
- net HM01B0_SDA: no longer SJ16.1
- net HM01B0_TRIG: no longer SJ4.1
- net HM01B0_VS: no longer SJ3.1
- net ICE40_+1V2_CORE: now also JP5.2; no longer JP20.2
- net ICE40_+1V2_PLL: now also JP6.2; no longer JP5.2
- net ICE40_GPIO43: no longer SJ17.1
- net ICE40_SPI_VCCIO1: now also JP8.2; no longer JP7.2
- net ICE40_VCCIO0: now also JP13.2; no longer JP8.2
- net ICE40_VCCIO2: now also JP20.2; no longer JP13.2
- net ICE40_VPP2V5_+3V3: now also JP7.2; no longer JP6.2
- net MEM1_!HOLD: now also U16.!HOLD!/DQ3, U17.!HOLD!/DQ3; no longer JP25.3, JP26.3
- net MEM1_!WP: now also U16.!WP!/DQ2, U17.!WP!/DQ2; no longer JP23.5, JP24.5
- net MEM1_CIPO: now also U16.SO/DQ1, U17.SO/DQ1; no longer JP23.3, JP24.3
- net MEM1_COPI: now also U16.SI/DQ0, U17.SI/DQ0; no longer JP25.7, JP26.7
- net MEM1_PS1: now also U16.!CS; no longer JP23.1
- net MEM1_PS2: now also U17.!CS; no longer JP24.1
- net MEM1_SCK: now also U16.SCK, U17.SCK; no longer JP25.5, JP26.5
- net MEM1_VCC1: now also C59.P$2, C60.P$2, JP23.2, U16.VCC; no longer JP25.1, JP31.2
- net MEM1_VCC2: now also C61.P$2, C62.P$2, JP24.2, U17.VCC; no longer JP26.1, JP32.2
- net MEM2_!WP: now also U14.!WP, U15.!WP; no longer JP27.5, JP28.5
- net MEM2_CIPO1: now also U14.SO; no longer JP27.3
- net MEM2_CIPO2: now also U15.SO; no longer JP28.3
- net MEM2_COPI1: now also U14.SI; no longer JP29.7
- net MEM2_COPI2: now also U15.SI; no longer JP30.7
- net MEM2_PS1: now also U14.!CS; no longer JP27.1
- net MEM2_PS2: now also U15.!CS; no longer JP28.1
- net MEM2_SCK: now also U14.SCK, U15.SCK; no longer JP29.5, JP30.5
- net MEM2_VCC1: now also C55.P$2, C57.P$2, JP25.2, JP26.2, U14.!HOLD, U14.VDD; no longer JP29.1, JP33.2, JP34.2
- net MEM2_VCC2: now also C56.P$2, C58.P$2, JP27.2, JP28.2, U15.!HOLD, U15.VDD; no longer JP30.1, JP35.2, JP36.2
- net MIC1_VCC: now also JP29.2; no longer JP37.2
- net MIC2_VCC: now also JP30.2; no longer JP38.2
- net N$22: now also JP1.2, R22.1; no longer JP3.2, R24.1
- net N$3: now also JP3.2, R24.1; no longer JP1.2, R22.1

Commit message: routing for pcbng variant wip
Parts:
- removed C27, C28, C30, C48: 22u, rcl:C-USC1210
- removed LED6: (no value), led:LEDCHIPLED_0603
- removed R36: 1k, milliLearn-ice40:R0402_COMPACT
- added JP31: (no value), pinhead:PINHD-1X2
- added TP0, TP1, TP10, TP11, TP12, TP13, TP14, TP15, TP16, TP17, TP18, TP2, TP3, TP4, TP5, TP6, TP7, TP8, TP9: TPTP10SQ, testpad:TPTP10SQ
Connections:
- removed net I2S_WS: JP40.29, U12.WS, U13.WS, U8.21
- removed net ICE40_GPIO4: JP41.15
- removed net N$32: LED4.A, R36.P$2
- new net I2S_DATA: JP40.25, U12.DATA, U13.DATA, U8.18
- new net N$34: U13.WS
- new net N$35: U13.BLK
- new net N$36: U12.BLK
- new net N$37: U12.WS
- net +1V2_METERED: now also C26.1, R24.2, U9.IN-1; no longer C24.1, C27.1, R22.2, U9.IN-3
- net +1V8_METERED: no longer C28.1
- net +2V8_METERED: no longer C48.1
- net +3V3: now also U13.SEL; no longer R36.P$1
- net +3V3_METERED: now also C24.1, R22.2, U9.IN-3; no longer C26.1, C30.1, R24.2, U9.IN-1
- net GND: now also JP31.2, LED5.C, TP0.TP, TP17.TP, TP18.TP; no longer C27.2, C28.2, C30.2, C48.2, LED6.C
- net HM01B0_D0: now also TP9.TP
- net HM01B0_D1: now also TP1.TP
- net HM01B0_D2: now also TP6.TP
- net HM01B0_D3: now also TP2.TP
- net HM01B0_D4: now also TP7.TP
- net HM01B0_D5: now also TP14.TP
- net HM01B0_D6: now also TP13.TP
- net HM01B0_D7: now also TP8.TP
- net HM01B0_HS: now also TP10.TP
- net HM01B0_INT: now also TP12.TP
- net HM01B0_MCK: now also TP5.TP
- net HM01B0_PCLK: now also TP11.TP
- net HM01B0_SCL: now also TP15.TP
- net HM01B0_SDA: now also TP16.TP
- net HM01B0_TRIG: now also LED4.C, TP4.TP; no longer LED5.C
- net HM01B0_VS: now also TP3.TP
- net ICE40_CRESETB: now also JP31.1
- net ICE40_FLASH_CIPO: now also JP40.9; no longer JP40.21, JP40.27, U12.DATA, U13.DATA
- net ICE40_FLASH_COPI: now also JP40.5; no longer JP40.15, LED4.C
- net ICE40_FLASH_PS: now also JP40.1; no longer JP40.19
- net ICE40_FLASH_SCK: now also JP40.3; no longer JP40.17, U12.BLK, U13.BLK
- net ICE40_GPIO43: now also LED5.A; no longer LED6.A
- net ICE40_OSC_12M: now also JP40.23; no longer JP41.1
- net MEM1_!HOLD: now also JP40.17, U8.10; no longer JP40.13, U8.13
- net MEM1_!WP: now also JP40.15, U8.7; no longer JP40.11, U8.12
- net MEM1_CIPO: now also JP40.7, U8.6; no longer JP40.9, U8.11
- net MEM1_COPI: now also JP40.21, U8.12; no longer JP40.25, U8.19
- net MEM1_PS1: now also JP40.11; no longer JP40.5
- net MEM1_PS2: now also JP40.13, U8.13; no longer JP40.7, U8.10
- net MEM1_SCK: now also JP40.19, U8.11; no longer JP40.23, U8.18
- net MEM2_!WP: now also U8.2; no longer JP41.9, U8.48
- net MEM2_CIPO1: now also U8.45; no longer JP41.7, U8.47
- net MEM2_CIPO2: now also U8.48; no longer U8.4
- net MEM2_COPI1: now also U8.46; no longer JP41.11, U8.2
- net MEM2_COPI2: now also U8.4; no longer U8.44
- net MEM2_PS1: now also U8.44; no longer JP41.3, U8.45
- net MEM2_PS2: now also U8.47; no longer JP41.5, U8.46
- net MEM2_SCK: no longer JP41.13
- net MIC2_VCC: no longer U13.SEL
- net N$33: now also LED4.A; no longer LED5.A
- net QWIIC_SCL: now also JP40.27, U8.21; no longer JP40.3, U8.7
- net QWIIC_SDA: now also JP40.29, U8.19; no longer JP40.1, U8.6
Other:
- moved on the sheet: LED5, R37

Commit message: first pass of routing done
Parts:
- C1: value (none) -> 1u; MFR (none) -> SAMSUNG; MFR_PN (none) -> CL05A105KO5NNNC
- C32, C38: MFR (none) -> SAMSUNG; MFR_PN (none) -> CL05B104KO5NNNC
- J1: MFR (none) -> AMPHENOL; MFR_PN (none) -> SFV24R-2STE1HLF
- J2: MFR (none) -> 10118194-0001LF; MFR_PN (none) -> 10118194-0001LF
- J3: MFR (none) -> JST; MFR_PN (none) -> SM04B-SRSS-TB(LF)(SN)
- R25: MFR (none) -> YAGEO; MFR_PN (none) -> RC0402FR-07100RL
- SW1, SW2: MFR (none) -> TE; MFR_PN (none) -> FSM4JSMATR
- U11, U2: MFR (none) -> MICROCHIP; MFR_PN (none) -> DSC6111CI2A-012.0000
- U14, U15: MFR (none) -> CYPRESS; MFR_PN (none) -> CY15B104Q-LHXI
- U16, U17: MFR (none) -> ADESTO; MFR_PN (none) -> AT25QF641B-SHB-T
- U5: MFR (none) -> FTDI; MFR_PN (none) -> FT232HQ
- U7: MFR (none) -> MICRON; MFR_PN (none) -> MT25QL128ABA1EW7-0SIT
- U8: MFR (none) -> LATTICE; MFR_PN (none) -> ICE40UP5K-SG48I
Connections:
- net N$23 renamed MEAS_1V2
- net N$24 renamed MEAS_1V8
- net N$25 renamed MEAS_3V3
- net N$26 renamed MEAS_2V8
- removed net N$34: U13.WS
- removed net N$35: U13.BLK
- removed net N$36: U12.BLK
- removed net N$37: U12.WS
- net ICE40_FLASH_CIPO: now also U12.WS, U13.WS
- net ICE40_FLASH_SCK: now also U12.BLK, U13.BLK
- net MEM2_!WP: now also JP41.5
- net MEM2_CIPO1: now also JP41.3
- net MEM2_CIPO2: now also JP41.11
- net MEM2_COPI1: now also JP41.7
- net MEM2_COPI2: now also JP41.15
- net MEM2_PS1: now also JP41.1
- net MEM2_PS2: now also JP41.9
- net MEM2_SCK: now also JP41.13

Commit message: fix hm01b0 connector footprint
Parts:
- U5: MFR_PN FT232HQ -> FT232HQ-REEL
Changed lines of the file:
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@@
 <setting verticaltext="up"/>
 </settings>
-<grid distance="0.05" unitdist="inch" unit="inch" style="lines" multiple="1" display="yes" altdistance="0.01" altunitdist="inch" altunit="inch"/>
+<grid distance="0.1" unitdist="inch" unit="inch" style="lines" multiple="1" display="no" altdistance="0.01" altunitdist="inch" altunit="inch"/>
 <layers>
-<layer number="1" name="Top" color="4" fill="1" visible="yes" active="no"/>
-<layer number="2" name="Route2" color="16" fill="10" visible="yes" active="no"/>
-<layer number="3" name="Route3" color="17" fill="1" visible="yes" active="no"/>
-<layer number="4" name="Route4" color="18" fill="1" visible="yes" active="no"/>
-<layer number="5" name="Route5" color="19" fill="1" visible="yes" active="no"/>
-<layer number="6" name="Route6" color="25" fill="1" visible="yes" active="no"/>
-<layer number="7" name="Route7" color="26" fill="1" visible="yes" active="no"/>
-<layer number="8" name="Route8" color="27" fill="1" visible="yes" active="no"/>
-<layer number="9" name="Route9" color="28" fill="1" visible="yes" active="no"/>
-<layer number="10" name="Route10" color="29" fill="1" visible="yes" active="no"/>
-<layer number="11" name="Route11" color="30" fill="1" visible="yes" active="no"/>
-<layer number="12" name="Route12" color="20" fill="1" visible="yes" active="no"/>
-<layer number="13" name="Route13" color="21" fill="1" visible="yes" active="no"/>
-<layer number="14" name="Route14" color="22" fill="1" visible="yes" active="no"/>
-<layer number="15" name="Route15" color="23" fill="11" visible="yes" active="no"/>
-<layer number="16" name="Bottom" color="1" fill="1" visible="yes" active="no"/>
-<layer number="17" name="Pads" color="2" fill="1" visible="yes" active="no"/>
-<layer number="18" name="Vias" color="2" fill="1" visible="yes" active="no"/>
-<layer number="19" name="Unrouted" color="6" fill="1" visible="yes" active="no"/>
-<layer number="20" name="Dimension" color="24" fill="1" visible="yes" active="no"/>
-<layer number="21" name="tPlace" color="7" fill="1" visible="yes" active="no"/>
-<layer number="22" name="bPlace" color="7" fill="1" visible="yes" active="no"/>
-<layer number="23" name="tOrigins" color="15" fill="1" visible="yes" active="no"/>
-<layer number="24" name="bOrigins" color="15" fill="1" visible="yes" active="no"/>
-<layer number="25" name="tNames" color="7" fill="1" visible="yes" active="no"/>
-<layer number="26" name="bNames" color="7" fill="1" visible="yes" active="no"/>
-<layer number="27" name="tValues" color="7" fill="1" visible="yes" active="no"/>
-<layer number="28" name="bValues" color="7" fill="1" visible="yes" active="no"/>
+<layer number="1" name="Top" color="4" fill="1" visible="no" active="no"/>
+<layer number="2" name="Route2" color="16" fill="10" visible="no" active="no"/>
+<layer number="3" name="Route3" color="17" fill="1" visible="no" active="no"/>
+<layer number="4" name="Route4" color="18" fill="1" visible="no" active="no"/>
+<layer number="5" name="Route5" color="19" fill="1" visible="no" active="no"/>
+<layer number="6" name="Route6" color="25" fill="1" visible="no" active="no"/>
+<layer number="7" name="Route7" color="26" fill="1" visible="no" active="no"/>
+<layer number="8" name="Route8" color="27" fill="1" visible="no" active="no"/>
+<layer number="9" name="Route9" color="28" fill="1" visible="no" active="no"/>
+<layer number="10" name="Route10" color="29" fill="1" visible="no" active="no"/>
+<layer number="11" name="Route11" color="30" fill="1" visible="no" active="no"/>
+<layer number="12" name="Route12" color="20" fill="1" visible="no" active="no"/>
+<layer number="13" name="Route13" color="21" fill="1" visible="no" active="no"/>
+<layer number="14" name="Route14" color="22" fill="1" visible="no" active="no"/>
+<layer number="15" name="Route15" color="23" fill="11" visible="no" active="no"/>
+<layer number="16" name="Bottom" color="1" fill="1" visible="no" active="no"/>
+<layer number="17" name="Pads" color="2" fill="1" visible="no" active="no"/>
+<layer number="18" name="Vias" color="2" fill="1" visible="no" active="no"/>
+<layer number="19" name="Unrouted" color="6" fill="1" visible="no" active="no"/>
+<layer number="20" name="Dimension" color="24" fill="1" visible="no" active="no"/>
+<layer number="21" name="tPlace" color="7" fill="1" visible="no" active="no"/>
+<layer number="22" name="bPlace" color="7" fill="1" visible="no" active="no"/>
+<layer number="23" name="tOrigins" color="15" fill="1" visible="no" active="no"/>
+<layer number="24" name="bOrigins" color="15" fill="1" visible="no" active="no"/>
+<layer number="25" name="tNames" color="7" fill="1" visible="no" active="no"/>
+<layer number="26" name="bNames" color="7" fill="1" visible="no" active="no"/>
+<layer number="27" name="tValues" color="7" fill="1" visible="no" active="no"/>
+<layer number="28" name="bValues" color="7" fill="1" visible="no" active="no"/>
 <layer number="29" name="tStop" color="7" fill="3" visible="no" active="no"/>
 <layer number="30" name="bStop" color="7" fill="6" visible="no" active="no"/>
@@
 <layer number="35" name="tGlue" color="7" fill="4" visible="no" active="no"/>
 <layer number="36" name="bGlue" color="7" fill="5" visible="no" active="no"/>
-<layer number="37" name="tTest" color="7" fill="1" visible="yes" active="no"/>
-<layer number="38" name="bTest" color="7" fill="1" visible="yes" active="no"/>
+<layer number="37" name="tTest" color="7" fill="1" visible="no" active="no"/>
+<layer number="38" name="bTest" color="7" fill="1" visible="no" active="no"/>
 <layer number="39" name="tKeepout" color="4" fill="11" visible="no" active="no"/>
 <layer number="40" name="bKeepout" color="1" fill="11" visible="no" active="no"/>
@@
 <layer number="44" name="Drills" color="7" fill="1" visible="no" active="no"/>
 <layer number="45" name="Holes" color="7" fill="1" visible="no" active="no"/>
-<layer number="46" name="Milling" color="3" fill="1" visible="yes" active="no"/>
-<layer number="47" name="Measures" color="7" fill="1" visible="yes" active="no"/>
-<layer number="48" name="Document" color="7" fill="1" visible="yes" active="no"/>
-<layer number="49" name="Reference" color="7" fill="1" visible="yes" active="no"/>
-<layer number="50" name="dxf" color="7" fill="1" visible="yes" active="no"/>
-<layer number="51" name="tDocu" color="7" fill="1" visible="yes" active="no"/>
-<layer number="52" name="bDocu" color="7" fill="1" visible="yes" active="no"/>
-<layer number="53" name="tGND_GNDA" color="7" fill="9" visible="yes" active="no"/>
-<layer number="54" name="bGND_GNDA" color="1" fill="9" visible="yes" active="no"/>
-<layer number="56" name="wert" color="7" fill="1" visible="yes" active="no"/>
-<layer number="57" name="tCAD" color="7" fill="1" visible="yes" active="no"/>
-<layer number="59" name="tCarbon" color="7" fill="1" visible="yes" active="no"/>
-<layer number="60" name="bCarbon" color="7" fill="1" visible="yes" active="no"/>
+<layer number="46" name="Milling" color="3" fill="1" visible="no" active="no"/>
+<layer number="47" name="Measures" color="7" fill="1" visible="no" active="no"/>
+<layer number="48" name="Document" color="7" fill="1" visible="no" active="no"/>
+<layer number="49" name="Reference" color="7" fill="1" visible="no" active="no"/>
+<layer number="50" name="dxf" color="7" fill="1" visible="no" active="no"/>
+<layer number="51" name="tDocu" color="7" fill="1" visible="no" active="no"/>
+<layer number="52" name="bDocu" color="7" fill="1" visible="no" active="no"/>
+<layer number="53" name="tGND_GNDA" color="7" fill="9" visible="no" active="no"/>
+<layer number="54" name="bGND_GNDA" color="1" fill="9" visible="no" active="no"/>
+<layer number="56" name="wert" color="7" fill="1" visible="no" active="no"/>
+<layer number="57" name="tCAD" color="7" fill="1" visible="no" active="no"/>
+<layer number="59" name="tCarbon" color="7" fill="1" visible="no" active="no"/>
+<layer number="60" name="bCarbon" color="7" fill="1" visible="no" active="no"/>
 <layer number="88" name="SimResults" color="9" fill="1" visible="yes" active="yes"/>
 <layer number="89" name="SimProbes" color="9" fill="1" visible="yes" active="yes"/>
@@
 <part name="U5" library="gtjennings_pcb_121217_1200_release" deviceset="MICROBUILDER_FT232H" device="Q">
 <attribute name="MFR" value="FTDI"/>
-<attribute name="MFR_PN" value="FT232HQ"/>
+<attribute name="MFR_PN" value="FT232HQ-REEL"/>
 </part>
 <part name="C4" library="milliLearn-ice40" deviceset="C0402_COMPACT" device="" value="100n">
